Commit message: feat: Add X12-150 URDF

File: myactuator_rmd_description/urdf/myactuator_rmd.ros2_control.xacro (robot description, xacro)
@@ -7,5 +7,4 @@
         <xacro:if value="${simulation}">
           <plugin>gazebo_ros2_control/GazeboSystem</plugin>
-          <!-- <plugin>fake_components/GenericActuator</plugin> -->
         </xacro:if>
         <xacro:unless value="${simulation}">

File: myactuator_rmd_description/urdf/myactuator_rmd.xacro (robot description, xacro)
@@ -77,5 +77,5 @@
       <child link="${name}_shaft" />
       <axis xyz="0 0 1"/>
-      <limit effort="87" lower="${-pi}" upper="${pi}" velocity="2.0"/>
+      <limit effort="80" lower="${-pi}" upper="${pi}" velocity="2.0"/>
     </joint>
     <joint name="${name}_to_${name}_shaft" type="fixed">
