Commit message: add timeout support

File: myactuator_rmd_description/urdf/X8ProV2.xacro (robot description, xacro)
@@ -7,4 +7,5 @@
                           ifname="${ifname}" actuator_id="${actuator_id}"
                           torque_constant="2.6"
+                          timeout="1000"
                           limit_effort="25.0" limit_lower="${-pi}" limit_upper="${pi}"
                           limit_velocity="${122/60*2*pi}"

File: myactuator_rmd_description/urdf/myactuator_rmd.ros2_control.xacro (robot description, xacro)
@@ -2,5 +2,5 @@
 <robot xmlns:xacro="http://www.ros.org/wiki/xacro">
   <!-- ros2_control configuration for a given joint -->
-  <xacro:macro name="myactuator_rmd_ros2_control" params="name joint_name simulation ifname actuator_id torque_constant">
+  <xacro:macro name="myactuator_rmd_ros2_control" params="name joint_name simulation ifname actuator_id torque_constant timeout">
     <ros2_control name="${name}" type="actuator">
       <hardware>
@@ -16,4 +16,6 @@
           <!-- Torque constant of the actuator -->
           <param name="torque_constant">${torque_constant}</param>
+          <!-- Timeout of the actuator -->
+          <param name="timeout">${timeout}</param>
         </xacro:unless>
       </hardware>

File: myactuator_rmd_description/urdf/myactuator_rmd.xacro (robot description, xacro)
@@ -17,4 +17,5 @@
                                              simulation ifname actuator_id
                                              torque_constant
+                                             timeout
                                              limit_effort limit_lower limit_upper
                                              limit_velocity
@@ -93,5 +94,5 @@
     <!-- ros2_control configuration -->
     <xacro:myactuator_rmd_ros2_control name="${prefix}${joint_name}_ros2_control" joint_name="${prefix}${joint_name}" simulation="${simulation}"
-                                       ifname="${ifname}" actuator_id="${actuator_id}" torque_constant="${torque_constant}"/>
+                                       ifname="${ifname}" actuator_id="${actuator_id}" torque_constant="${torque_constant}" timeout="${timeout}"/>
   </xacro:macro>
 </robot>
