Commit message: refactor: Modify URDF structure and naming conventions

File: myactuator_rmd_description/urdf/X12_150.xacro (robot description, xacro)
@@ -3,7 +3,6 @@
   <xacro:include filename="$(find myactuator_rmd_description)/urdf/myactuator_rmd.xacro"/>
   <!-- Provide dimensions for specific actuator -->
-  <xacro:macro name="X12_150" params="name parent_link child_link joint_name simulation ifname actuator_id">
-    <xacro:myactuator_rmd name="${name}" parent_link="${parent_link}" child_link="${child_link}"
-                          joint_name="${joint_name}" simulation="${simulation}"
+  <xacro:macro name="X12_150" params="prefix joint_name simulation ifname actuator_id">
+    <xacro:myactuator_rmd prefix="${prefix}" joint_name="${joint_name}" simulation="${simulation}"
                           ifname="${ifname}" actuator_id="${actuator_id}"
                           visual="$(find myactuator_rmd_description)/meshes/visual/X12_150/X12_150.dae"

File: myactuator_rmd_description/urdf/X8ProV2.xacro (robot description, xacro)
@@ -3,7 +3,6 @@
   <xacro:include filename="$(find myactuator_rmd_description)/urdf/myactuator_rmd.xacro"/>
   <!-- Provide dimensions for specific actuator -->
-  <xacro:macro name="X8ProV2" params="name parent_link child_link joint_name simulation ifname actuator_id">
-    <xacro:myactuator_rmd name="${name}" parent_link="${parent_link}" child_link="${child_link}"
-                          joint_name="${joint_name}" simulation="${simulation}"
+  <xacro:macro name="X8ProV2" params="prefix joint_name simulation ifname actuator_id">
+    <xacro:myactuator_rmd prefix="${prefix}" joint_name="${joint_name}" simulation="${simulation}"
                           ifname="${ifname}" actuator_id="${actuator_id}"
                           visual="$(find myactuator_rmd_description)/meshes/visual/X8ProV2/X8ProV2.dae"

File: myactuator_rmd_description/urdf/myactuator_rmd.xacro (robot description, xacro)
@@ -9,11 +9,12 @@
       <origin xyz="${x} ${y} ${z}" rpy="0 0 0"/>
       <inertia ixx="${1/12*m*height*height}" ixy="0.0" ixz="0.0"
-                iyy="${1/12*m*height*height}" iyz="0.0"
-                izz="${1/2*m*radius*radius}"/>
+               iyy="${1/12*m*height*height}" iyz="0.0"
+               izz="${1/2*m*radius*radius}"/>
     </inertial>
   </xacro:macro>
   <!-- Actuator geometry -->
-  <xacro:macro name="myactuator_rmd" params="name parent_link child_link joint_name
-                                             simulation ifname actuator_id visual
+  <xacro:macro name="myactuator_rmd" params="prefix joint_name
+                                             simulation ifname actuator_id
+                                             visual
                                              radius_1 height_1
                                              radius_2 height_2
@@ -27,5 +28,5 @@
     <xacro:property name="mass_2" value="${volume_2/volume_1_2_3*mass}"/>
     <xacro:property name="mass_3" value="${volume_3/volume_1_2_3*mass}"/>
-    <link name="${name}">
+    <link name="${prefix}actuator_backplate">
       <visual>
         <geometry>
@@ -42,10 +43,5 @@
                                radius="${radius_1}" height="${height_1}"/>
     </link>
-    <joint name="${parent_link}_to_${name}" type="fixed">
-      <origin xyz="0 0 0" rpy="0 0 0" />
-      <parent link="${parent_link}" />
-      <child link="${name}" />
-    </joint>
-    <link name="${name}_body">
+    <link name="${prefix}actuator_back_flange">
       <collision>
         <origin xyz="0 0 ${height_2/2}" rpy="0 0 0"/>
@@ -57,10 +53,16 @@
                                radius="${radius_2}" height="${height_2}"/>
     </link>
-    <joint name="${name}_to_${name}_body" type="fixed">
+    <joint name="${prefix}actuator_backplate_to_${prefix}actuator_back_flange" type="fixed">
       <origin xyz="0 0 ${height_1}" rpy="0 0 0" />
-      <parent link="${name}" />
-      <child link="${name}_body" />
+      <parent link="${prefix}actuator_backplate" />
+      <child link="${prefix}actuator_back_flange" />
     </joint>
-    <link name="${name}_shaft">
+    <link name="${prefix}actuator_front_flange"/>
+    <joint name="${prefix}actuator_back_flange_to_${prefix}actuator_front_flange" type="fixed">
+      <origin xyz="0 0 ${height_2}" rpy="0 0 0" />
+      <parent link="${prefix}actuator_back_flange" />
+      <child link="${prefix}actuator_front_flange" />
+    </joint>
+    <link name="${prefix}actuator_shaft">
       <collision>
         <origin xyz="0 0 ${height_3/2}" rpy="0 0 0"/>
@@ -72,18 +74,20 @@
                                radius="${radius_3}" height="${height_3}"/>
     </link>
-    <joint name="${joint_name}" type="revolute">
+    <!-- Joint has to be mounted to links with inertial properties  -->
+    <joint name="${prefix}${joint_name}" type="revolute">
       <origin xyz="0 0 ${height_2}" rpy="0 0 0" />
-      <parent link="${name}_body" />
-      <child link="${name}_shaft" />
+      <parent link="${prefix}actuator_back_flange" />
+      <child link="${prefix}actuator_shaft" />
       <axis xyz="0 0 1"/>
       <limit effort="80" lower="${-pi}" upper="${pi}" velocity="2.0"/>
     </joint>
-    <joint name="${name}_to_${name}_shaft" type="fixed">
+    <link name="${prefix}actuator_shaft_flange"/>
+    <joint name="${prefix}actuator_shaft_to_${prefix}actuator_shaft_flange" type="fixed">
       <origin xyz="0 0 ${height_3}" rpy="0 0 0" />
-      <parent link="${name}_shaft" />
-      <child link="${child_link}" />
+      <parent link="${prefix}actuator_shaft" />
+      <child link="${prefix}actuator_shaft_flange" />
     </joint>
     <!-- ros2_control configuration -->
-    <xacro:myactuator_rmd_ros2_control name="${joint_name}_ros2_control" joint_name="${joint_name}" simulation="${simulation}"
+    <xacro:myactuator_rmd_ros2_control name="${prefix}${joint_name}_ros2_control" joint_name="${prefix}${joint_name}" simulation="${simulation}"
                                        ifname="${ifname}" actuator_id="${actuator_id}"/>
   </xacro:macro>

File: myactuator_rmd_description/urdf/standalone.urdf.xacro (robot description, xacro)
@@ -1,4 +1,6 @@
 <?xml version="1.0"?>
 <robot xmlns:xacro="http://www.ros.org/wiki/xacro" name="myactuator_rmd">
+  <!-- Prefix for multiple actuators in the same URDF -->
+  <xacro:arg name="prefix" default=""/>
   <!-- Model of the actuator to be used -->
   <xacro:arg name="actuator" default="X8ProV2"/>
@@ -13,12 +15,9 @@
   <xacro:property name="child_link" value="child"/>
   <xacro:property name="joint_name" value="joint"/>
-  <!-- Parent and child link -->
-  <link name="${parent_link}"/>
-  <link name="${child_link}"/>
   <!-- Actuator -->
   <xacro:property name="actuator_model" value="$(arg actuator)"/>
   <xacro:if value="${actuator_model == 'X8ProV2'}">
     <xacro:include filename="$(find myactuator_rmd_description)/urdf/X8ProV2.xacro"/>
-    <xacro:X8ProV2 name="X8ProV2" parent_link="${parent_link}" child_link="${child_link}" joint_name="${joint_name}"
+    <xacro:X8ProV2 prefix="$(arg prefix)" joint_name="${joint_name}"
                    simulation="$(arg simulation)"
                    ifname="$(arg ifname)" actuator_id="$(arg actuator_id)"/>
@@ -26,8 +25,21 @@
   <xacro:if value="${actuator_model == 'X12_150'}">
     <xacro:include filename="$(find myactuator_rmd_description)/urdf/X12_150.xacro"/>
-    <xacro:X12_150 name="X12_150" parent_link="${parent_link}" child_link="${child_link}" joint_name="${joint_name}"
+    <xacro:X12_150 prefix="$(arg prefix)" joint_name="${joint_name}"
                    simulation="$(arg simulation)"
                    ifname="$(arg ifname)" actuator_id="$(arg actuator_id)"/>
   </xacro:if>
+  <!-- Parent and child link and their fixed joints to the actuator -->
+  <link name="${parent_link}"/>
+  <link name="${child_link}"/>
+  <joint name="${parent_link}_to_actuator" type="fixed">
+    <origin xyz="0 0 0" rpy="0 0 0" />
+    <parent link="${parent_link}" />
+    <child link="$(arg prefix)actuator_backplate" />
+  </joint>
+  <joint name="actuator_to_${child_link}" type="fixed">
+    <origin xyz="0 0 0" rpy="0 0 0" />
+    <parent link="$(arg prefix)actuator_shaft_flange" />
+    <child link="${child_link}" />
+  </joint>
   <!-- Gazebo ros2_control plug-in -->
   <xacro:if value="$(arg simulation)">

Commit message: refactor: Update Xacro files with new parameters and update documentation

File: myactuator_rmd_description/urdf/X12_150.xacro (robot description, xacro)
@@ -6,4 +6,7 @@
     <xacro:myactuator_rmd prefix="${prefix}" joint_name="${joint_name}" simulation="${simulation}"
                           ifname="${ifname}" actuator_id="${actuator_id}"
+                          torque_constant="3.33"
+                          limit_effort="150.0" limit_lower="${-pi}" limit_upper="${pi}"
+                          limit_velocity="${100/60*2*pi}"
                           visual="$(find myactuator_rmd_description)/meshes/visual/X12_150/X12_150.dae"
                           radius_1="0.04"  height_1="0.0136"

File: myactuator_rmd_description/urdf/X8ProV2.xacro (robot description, xacro)
@@ -6,4 +6,7 @@
     <xacro:myactuator_rmd prefix="${prefix}" joint_name="${joint_name}" simulation="${simulation}"
                           ifname="${ifname}" actuator_id="${actuator_id}"
+                          torque_constant="2.6"
+                          limit_effort="25.0" limit_lower="${-pi}" limit_upper="${pi}"
+                          limit_velocity="${122/60*2*pi}"
                           visual="$(find myactuator_rmd_description)/meshes/visual/X8ProV2/X8ProV2.dae"
                           radius_1="0.028" height_1="0.0125"

File: myactuator_rmd_description/urdf/myactuator_rmd.ros2_control.xacro (robot description, xacro)
@@ -2,5 +2,5 @@
 <robot xmlns:xacro="http://www.ros.org/wiki/xacro">
   <!-- ros2_control configuration for a given joint -->
-  <xacro:macro name="myactuator_rmd_ros2_control" params="name joint_name simulation ifname actuator_id">
+  <xacro:macro name="myactuator_rmd_ros2_control" params="name joint_name simulation ifname actuator_id torque_constant">
     <ros2_control name="${name}" type="actuator">
       <hardware>
@@ -10,15 +10,19 @@
         <xacro:unless value="${simulation}">
           <plugin>myactuator_rmd_hardware/MyActuatorRmdHardwareInterface</plugin>
+          <!-- The name of the CAN interface -->
           <param name="ifname">${ifname}</param>
+          <!-- The id used for the CAN communication -->
           <param name="actuator_id">${actuator_id}</param>
+          <!-- Torque constant of the actuator -->
+          <param name="torque_constant">${torque_constant}</param>
         </xacro:unless>
       </hardware>
       <joint name="${joint_name}">
+        <command_interface name="position"/>
+        <command_interface name="velocity"/>
         <command_interface name="effort"/>
-        <command_interface name="velocity"/>
-        <command_interface name="position"/>
+        <state_interface name="position"/>
+        <state_interface name="velocity"/>
         <state_interface name="effort"/>
-        <state_interface name="velocity"/>
-        <state_interface name="position"/>
       </joint>
     </ros2_control>

File: myactuator_rmd_description/urdf/myactuator_rmd.xacro (robot description, xacro)
@@ -16,4 +16,7 @@
   <xacro:macro name="myactuator_rmd" params="prefix joint_name
                                              simulation ifname actuator_id
+                                             torque_constant
+                                             limit_effort limit_lower limit_upper
+                                             limit_velocity
                                              visual
                                              radius_1 height_1
@@ -80,5 +83,5 @@
       <child link="${prefix}actuator_shaft" />
       <axis xyz="0 0 1"/>
-      <limit effort="80" lower="${-pi}" upper="${pi}" velocity="2.0"/>
+      <limit effort="${limit_effort}" lower="${limit_lower}" upper="${limit_upper}" velocity="${limit_velocity}"/>
     </joint>
     <link name="${prefix}actuator_shaft_flange"/>
@@ -90,5 +93,5 @@
     <!-- ros2_control configuration -->
     <xacro:myactuator_rmd_ros2_control name="${prefix}${joint_name}_ros2_control" joint_name="${prefix}${joint_name}" simulation="${simulation}"
-                                       ifname="${ifname}" actuator_id="${actuator_id}"/>
+                                       ifname="${ifname}" actuator_id="${actuator_id}" torque_constant="${torque_constant}"/>
   </xacro:macro>
 </robot>

Commit message: Implement extra thread for reading 0x9A and 0x9D (currently failing due to concurrent access to CAN resource)

File: myactuator_rmd_description/urdf/X12_150.xacro (robot description, xacro)
@@ -6,4 +6,5 @@
     <xacro:myactuator_rmd prefix="${prefix}" joint_name="${joint_name}" simulation="${simulation}"
                           ifname="${ifname}" actuator_id="${actuator_id}"
+                          extra_status_refresh_rate="${extra_status_refresh_rate}"
                           torque_constant="3.33"
                           limit_effort="150.0" limit_lower="${-pi}" limit_upper="${pi}"

File: myactuator_rmd_description/urdf/X8ProV2.xacro (robot description, xacro)
@@ -3,7 +3,8 @@
   <xacro:include filename="$(find myactuator_rmd_description)/urdf/myactuator_rmd.xacro"/>
   <!-- Provide dimensions for specific actuator -->
-  <xacro:macro name="X8ProV2" params="prefix joint_name simulation ifname actuator_id">
+  <xacro:macro name="X8ProV2" params="prefix joint_name simulation ifname actuator_id extra_status_refresh_rate">
     <xacro:myactuator_rmd prefix="${prefix}" joint_name="${joint_name}" simulation="${simulation}"
                           ifname="${ifname}" actuator_id="${actuator_id}"
+                          extra_status_refresh_rate="${extra_status_refresh_rate}"
                           torque_constant="2.6"
                           limit_effort="25.0" limit_lower="${-pi}" limit_upper="${pi}"

File: myactuator_rmd_description/urdf/myactuator_rmd.ros2_control.xacro (robot description, xacro)
@@ -2,5 +2,5 @@
 <robot xmlns:xacro="http://www.ros.org/wiki/xacro">
   <!-- ros2_control configuration for a given joint -->
-  <xacro:macro name="myactuator_rmd_ros2_control" params="name joint_name simulation ifname actuator_id torque_constant">
+  <xacro:macro name="myactuator_rmd_ros2_control" params="name joint_name simulation ifname actuator_id torque_constant extra_status_refresh_rate">
     <ros2_control name="${name}" type="actuator">
       <hardware>
@@ -16,4 +16,6 @@
           <!-- Torque constant of the actuator -->
           <param name="torque_constant">${torque_constant}</param>
+          <!-- Extra status refresh of the actuator -->
+          <param name="extra_status_refresh_rate">${extra_status_refresh_rate}</param>
         </xacro:unless>
       </hardware>

File: myactuator_rmd_description/urdf/myactuator_rmd.xacro (robot description, xacro)
@@ -17,4 +17,5 @@
                                              simulation ifname actuator_id
                                              torque_constant
+                                             extra_status_refresh_rate
                                              limit_effort limit_lower limit_upper
                                              limit_velocity
@@ -93,5 +94,5 @@
     <!-- ros2_control configuration -->
     <xacro:myactuator_rmd_ros2_control name="${prefix}${joint_name}_ros2_control" joint_name="${prefix}${joint_name}" simulation="${simulation}"
-                                       ifname="${ifname}" actuator_id="${actuator_id}" torque_constant="${torque_constant}"/>
+                                       ifname="${ifname}" actuator_id="${actuator_id}" torque_constant="${torque_constant}" extra_status_refresh_rate="${extra_status_refresh_rate}"/>
   </xacro:macro>
 </robot>

File: myactuator_rmd_description/urdf/standalone.urdf.xacro (robot description, xacro)
@@ -11,4 +11,6 @@
   <!-- CAN id for real hardware interface -->
   <xacro:arg name="actuator_id" default=""/>
+  <!-- Use for Extra Status Motor -->
+  <xacro:arg name="extra_status_refresh_rate" default="0"/>
   <!-- Define link names -->
   <xacro:property name="parent_link" value="world"/>
@@ -21,5 +23,6 @@
     <xacro:X8ProV2 prefix="$(arg prefix)" joint_name="${joint_name}"
                    simulation="$(arg simulation)"
-                   ifname="$(arg ifname)" actuator_id="$(arg actuator_id)"/>
+                   ifname="$(arg ifname)" actuator_id="$(arg actuator_id)"
+                   extra_status_refresh_rate="$(arg extra_status_refresh_rate)"/>
   </xacro:if>
   <xacro:if value="${actuator_model == 'X12_150'}">
@@ -27,5 +30,6 @@
     <xacro:X12_150 prefix="$(arg prefix)" joint_name="${joint_name}"
                    simulation="$(arg simulation)"
-                   ifname="$(arg ifname)" actuator_id="$(arg actuator_id)"/>
+                   ifname="$(arg ifname)" actuator_id="$(arg actuator_id)"
+                   extra_status_refresh_rate="$(arg extra_status_refresh_rate)"/>
   </xacro:if>
   <!-- Parent and child link and their fixed joints to the actuator -->

Commit message: feat: Add optional low-pass filter for torque

File: myactuator_rmd_description/urdf/X12_150.xacro (robot description, xacro)
@@ -6,4 +6,5 @@
     <xacro:myactuator_rmd prefix="${prefix}" joint_name="${joint_name}" simulation="${simulation}"
                           ifname="${ifname}" actuator_id="${actuator_id}"
+                          velocity_alpha="0.1" effort_alpha="0.1"
                           torque_constant="3.33"
                           limit_effort="150.0" limit_lower="${-pi}" limit_upper="${pi}"

File: myactuator_rmd_description/urdf/X8ProV2.xacro (robot description, xacro)
@@ -6,4 +6,5 @@
     <xacro:myactuator_rmd prefix="${prefix}" joint_name="${joint_name}" simulation="${simulation}"
                           ifname="${ifname}" actuator_id="${actuator_id}"
+                          velocity_alpha="0.1" effort_alpha="0.1"
                           torque_constant="2.6"
                           limit_effort="25.0" limit_lower="${-pi}" limit_upper="${pi}"

File: myactuator_rmd_description/urdf/myactuator_rmd.ros2_control.xacro (robot description, xacro)
@@ -2,5 +2,6 @@
 <robot xmlns:xacro="http://www.ros.org/wiki/xacro">
   <!-- ros2_control configuration for a given joint -->
-  <xacro:macro name="myactuator_rmd_ros2_control" params="name joint_name simulation ifname actuator_id torque_constant">
+  <xacro:macro name="myactuator_rmd_ros2_control" params="name joint_name simulation ifname actuator_id
+                                                          velocity_alpha effort_alpha torque_constant">
     <ros2_control name="${name}" type="actuator">
       <hardware>
@@ -16,4 +17,8 @@
           <!-- Torque constant of the actuator -->
           <param name="torque_constant">${torque_constant}</param>
+          <!-- Low-pass filter constant for velocity -->
+          <param name="velocity_alpha">${velocity_alpha}</param>
+          <!-- Low-pass filter constant for effort -->
+          <param name="effort_alpha">${effort_alpha}</param>
         </xacro:unless>
       </hardware>

File: myactuator_rmd_description/urdf/myactuator_rmd.xacro (robot description, xacro)
@@ -16,4 +16,5 @@
   <xacro:macro name="myactuator_rmd" params="prefix joint_name
                                              simulation ifname actuator_id
+                                             velocity_alpha:=0.1 effort_alpha:=0.1
                                              torque_constant
                                              limit_effort limit_lower limit_upper
@@ -93,5 +94,7 @@
     <!-- ros2_control configuration -->
     <xacro:myactuator_rmd_ros2_control name="${prefix}${joint_name}_ros2_control" joint_name="${prefix}${joint_name}" simulation="${simulation}"
-                                       ifname="${ifname}" actuator_id="${actuator_id}" torque_constant="${torque_constant}"/>
+                                       ifname="${ifname}" actuator_id="${actuator_id}"
+                                       velocity_alpha="${velocity_alpha}" effort_alpha="${effort_alpha}"
+                                       torque_constant="${torque_constant}"/>
   </xacro:macro>
 </robot>
