Commit message: Add timeout parameter

File: myactuator_rmd_description/urdf/X12_150.xacro (robot description, xacro)
@@ -3,9 +3,10 @@
   <xacro:include filename="$(find myactuator_rmd_description)/urdf/myactuator_rmd.xacro"/>
   <!-- Provide dimensions for specific actuator -->
-  <xacro:macro name="X12_150" params="prefix joint_name simulation ifname actuator_id">
+  <xacro:macro name="X12_150" params="prefix joint_name simulation ifname actuator_id timeour">
     <xacro:myactuator_rmd prefix="${prefix}" joint_name="${joint_name}" simulation="${simulation}"
                           ifname="${ifname}" actuator_id="${actuator_id}"
                           velocity_alpha="0.1" effort_alpha="0.1"
                           torque_constant="3.33"
+                          timeout="${timeout}"
                           limit_effort="150.0" limit_lower="${-pi}" limit_upper="${pi}"
                           limit_velocity="${100/60*2*pi}"

File: myactuator_rmd_description/urdf/X8ProV2.xacro (robot description, xacro)
@@ -3,10 +3,10 @@
   <xacro:include filename="$(find myactuator_rmd_description)/urdf/myactuator_rmd.xacro"/>
   <!-- Provide dimensions for specific actuator -->
-  <xacro:macro name="X8ProV2" params="prefix joint_name simulation ifname actuator_id">
+  <xacro:macro name="X8ProV2" params="prefix joint_name simulation ifname actuator_id timeout">
     <xacro:myactuator_rmd prefix="${prefix}" joint_name="${joint_name}" simulation="${simulation}"
                           ifname="${ifname}" actuator_id="${actuator_id}"
                           velocity_alpha="0.1" effort_alpha="0.1"
                           torque_constant="2.6"
-                          timeout="1000"
+                          timeout="${timeout}"
                           limit_effort="25.0" limit_lower="${-pi}" limit_upper="${pi}"
                           limit_velocity="${122/60*2*pi}"

File: myactuator_rmd_description/urdf/myactuator_rmd.ros2_control.xacro (robot description, xacro)
@@ -3,5 +3,6 @@
   <!-- ros2_control configuration for a given joint -->
   <xacro:macro name="myactuator_rmd_ros2_control" params="name joint_name simulation ifname actuator_id
-                                                          velocity_alpha effort_alpha torque_constant timeout">
+                                                          velocity_alpha effort_alpha
+                                                          torque_constant timeout">
     <ros2_control name="${name}" type="actuator">
       <hardware>

File: myactuator_rmd_description/urdf/standalone.urdf.xacro (robot description, xacro)
@@ -11,4 +11,6 @@
   <!-- CAN id for real hardware interface -->
   <xacro:arg name="actuator_id" default=""/>
+  <!-- Timeout duration for the actuator operation -->
+  <xacro:arg name="timeout" default="0"/>
   <!-- Define link names -->
   <xacro:property name="parent_link" value="world"/>
@@ -21,5 +23,6 @@
     <xacro:X8ProV2 prefix="$(arg prefix)" joint_name="${joint_name}"
                    simulation="$(arg simulation)"
-                   ifname="$(arg ifname)" actuator_id="$(arg actuator_id)"/>
+                   ifname="$(arg ifname)" actuator_id="$(arg actuator_id)"
+                   timeout="$(arg timeout)"/>
   </xacro:if>
   <xacro:if value="${actuator_model == 'X12_150'}">
@@ -27,5 +30,6 @@
     <xacro:X12_150 prefix="$(arg prefix)" joint_name="${joint_name}"
                    simulation="$(arg simulation)"
-                   ifname="$(arg ifname)" actuator_id="$(arg actuator_id)"/>
+                   ifname="$(arg ifname)" actuator_id="$(arg actuator_id)"
+                   timeout="$(arg timeout)"/>
   </xacro:if>
   <!-- Parent and child link and their fixed joints to the actuator -->

Commit message: fix typo

File: myactuator_rmd_description/urdf/X12_150.xacro (robot description, xacro)
@@ -3,5 +3,5 @@
   <xacro:include filename="$(find myactuator_rmd_description)/urdf/myactuator_rmd.xacro"/>
   <!-- Provide dimensions for specific actuator -->
-  <xacro:macro name="X12_150" params="prefix joint_name simulation ifname actuator_id timeour">
+  <xacro:macro name="X12_150" params="prefix joint_name simulation ifname actuator_id timeout">
     <xacro:myactuator_rmd prefix="${prefix}" joint_name="${joint_name}" simulation="${simulation}"
                           ifname="${ifname}" actuator_id="${actuator_id}"
